File: AidonBoard32.kicad_pcb (KiCad board)
At the start: 2 copper layers, 49 x 63.3 mm, 31 parts, among them J1 RJ12, M1 MICRO_USB_18_TH, Q1 S8050, Q2 S8050, U1 AMS1117-3V3, U2 CP2102N-GQFN24, U3 ESP32-WROOM, U4 74HC04D

Commit message: Finished first revision of AidonBoard32!
Parts:
- added D6: 1N5819, Diode_SMD:D_SOD-123F, F.Cu at (105.2, 83.1)
- added G2: LOGO, Harry:Harry_3, F.Cu at (119.6, 41.7)
- C1, C10, C2, C3, C4, C5, C6, C7, C8, C9: footprint Capacitor_SMD:C_0603_1608Metric_Pad1.08x0.95mm_HandSolder -> Capacitor_SMD:C_1206_3216Metric_Pad1.33x1.80mm_HandSolder
- D1: value 1N5819/SS14 -> 1N5819
- R1, R2, R3, R4, R5, R6, R7: footprint Resistor_SMD:R_0603_1608Metric_Pad0.98x0.95mm_HandSolder -> Resistor_SMD:R_1206_3216Metric_Pad1.30x1.75mm_HandSolder
- U4: footprint Package_SO:SO-14_3.9x8.65mm_P1.27mm -> Package_SO:SOIC-14_3.9x8.7mm_P1.27mm
- moved R6 33.9 mm to (122.2, 57.9)
- moved Q2 33.7 mm to (118.9, 57.7)
- moved R4 27.6 mm to (89.0, 49.5), turned to 270 degrees
- moved D3 23.8 mm to (112.5, 55.4), turned to 0 degrees
- moved R3 21.8 mm to (112.3, 59.2), turned to 0 degrees
- moved D4 16.8 mm to (84.5, 49.5)
- moved R2 13.1 mm to (92.5, 59.1), turned to 0 degrees
- moved D2 11.5 mm to (92.5, 55.4), turned to 180 degrees
- moved C7 8.02 mm to (102.4, 56.9)
- moved U2 7.51 mm to (92.7, 65.9)
- moved C4 7.18 mm to (85.6, 65.9), turned to 270 degrees
- moved C3 6.57 mm to (82.2, 65.9), turned to 270 degrees
- moved R1 5.56 mm to (92.7, 72.4), turned to 180 degrees
- moved C2 5.53 mm to (96.0, 79.2), turned to 90 degrees
- moved Q1 5.33 mm to (82.3, 57.7), turned to 90 degrees
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Connections:
- net /UART_TX renamed Net-(U3-Pad28)
- C1 pad 1: VBUS -> +5V
- C7 pad 2: VBUS -> +5V
- D1 pad 1: VBUS -> +5V
- D1 pad 2: Net-(D1-Pad2) -> VBUS
- D5 pad 1: VBUS -> +5V
- J1 pad 1: Net-(J1-Pad1) -> VDD
- J1 pad 2: Net-(J1-Pad2) -> VDD
- J1 pad 5: Net-(J1-Pad5) -> /HAN_OUT
- J1 pad 6: Net-(J1-Pad6) -> GND
- M1 pad 1: Net-(D1-Pad2) -> VBUS
- U1 pad 3: VBUS -> +5V
- U4 pad 1: Net-(U4-Pad1) -> /HAN_OUT
- U4 pad 14: Net-(U4-Pad14) -> VDD
- U4 pad 2: Net-(U4-Pad2) -> /UART_RX
Routing:
- net +3V3: track 0.00 -> 159.2 mm, vias 0 -> 2
- net /D+: track 0.00 -> 63.1 mm
- net /D-: track 0.00 -> 60.8 mm
- net +5V: track 0.00 -> 59.0 mm
- net /RTS: track 0.00 -> 43.4 mm, vias 0 -> 3
- net VBUS: track 0.00 -> 43.0 mm
- net /DTR: track 0.00 -> 41.8 mm, vias 0 -> 3
- net /EN: track 0.00 -> 38.4 mm
- net /MCU_RX: track 0.00 -> 36.5 mm, vias 0 -> 2
- net /MCU_TX: track 0.00 -> 35.4 mm, vias 0 -> 2
- net GND: track 0.00 -> 28.2 mm
- net /UART_RX: track 0.00 -> 27.7 mm
- net VDD: track 0.00 -> 27.6 mm
- net /LED_RX: track 0.00 -> 21.0 mm
- net /LED_TX: track 0.00 -> 21.0 mm
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- added copper zone on B.Cu, net GND
- added copper zone on F.Cu, net GND

Commit message: Update
Parts:
- removed U4: 74HC04D, Package_SO:SOIC-14_3.9x8.7mm_P1.27mm
- added Q3: MMBT3904, Package_TO_SOT_SMD:SOT-23_Handsoldering, F.Cu at (85.5, 56.0)
- added Q4: MMBT3904, Package_TO_SOT_SMD:SOT-23_Handsoldering, F.Cu at (120.0, 45.5)
- added R10: 10K, Resistor_SMD:R_0603_1608Metric_Pad0.98x0.95mm_HandSolder, F.Cu at (120.1, 51.4)
- added R11: 1K, Resistor_SMD:R_0603_1608Metric_Pad0.98x0.95mm_HandSolder, F.Cu at (123.5, 50.0)
- added R12: 10K, Resistor_SMD:R_0603_1608Metric_Pad0.98x0.95mm_HandSolder, F.Cu at (116.5, 50.0)
- added R8: 220, Resistor_SMD:R_0603_1608Metric_Pad0.98x0.95mm_HandSolder, F.Cu at (116.5, 55.0)
- added R9: 220, Resistor_SMD:R_0603_1608Metric_Pad0.98x0.95mm_HandSolder, F.Cu at (123.5, 54.9)
- C10: value 10uF -> 0.1uF; footprint Capacitor_SMD:C_1206_3216Metric_Pad1.33x1.80mm_HandSolder -> Capacitor_SMD:C_0603_1608Metric_Pad1.08x0.95mm_HandSolder
- C4, C6: footprint Capacitor_SMD:C_1206_3216Metric_Pad1.33x1.80mm_HandSolder -> Capacitor_SMD:C_0603_1608Metric_Pad1.08x0.95mm_HandSolder
- C7: value 0.1uF -> 10uF
- C8: value 47uF -> 0.1uF; footprint Capacitor_SMD:C_1206_3216Metric_Pad1.33x1.80mm_HandSolder -> Capacitor_SMD:C_0603_1608Metric_Pad1.08x0.95mm_HandSolder
- C9: value 0.1uF -> 1uF
- D1: value 1N5819 -> SS54; footprint Diode_SMD:D_SOD-123F -> Diode_SMD:D_SMA
- D2, D3, D4: footprint LED_SMD:LED_1206_3216Metric_Pad1.42x1.75mm_HandSolder -> LED_SMD:LED_0603_1608Metric_Pad1.05x0.95mm_HandSolder
- D5: value WS2812B -> LED_Small; footprint LED_SMD:LED_WS2812B_PLCC4_5.0x5.0mm_P3.2mm -> LED_SMD:LED_0603_1608Metric_Pad1.05x0.95mm_HandSolder
- D6: value 1N5819 -> WS2812B; footprint Diode_SMD:D_SOD-123F -> LED_SMD:LED_WS2812B_PLCC4_5.0x5.0mm_P3.2mm
- J1: footprint Henrik-Connectors:RJ11-6 -> 5555165-1:TE_5555165-1
- M1: value MICRO_USB_18_TH -> U-F-M5DD-Y-L
- Q1: value S8050 -> Si2301CDS-T1-GE3
- Q2: value S8050 -> MMBT3904
- R1: value 1k -> 100K; footprint Resistor_SMD:R_1206_3216Metric_Pad1.30x1.75mm_HandSolder -> Resistor_SMD:R_0603_1608Metric_Pad0.98x0.95mm_HandSolder
- R2: value 1k -> 1K; footprint Resistor_SMD:R_1206_3216Metric_Pad1.30x1.75mm_HandSolder -> Resistor_SMD:R_0603_1608Metric_Pad0.98x0.95mm_HandSolder
- R3, R4: value 1k -> 10K; footprint Resistor_SMD:R_1206_3216Metric_Pad1.30x1.75mm_HandSolder -> Resistor_SMD:R_0603_1608Metric_Pad0.98x0.95mm_HandSolder
- R5: value 12k -> 10K; footprint Resistor_SMD:R_1206_3216Metric_Pad1.30x1.75mm_HandSolder -> Resistor_SMD:R_0603_1608Metric_Pad0.98x0.95mm_HandSolder
- R6: value 12k -> 220; footprint Resistor_SMD:R_1206_3216Metric_Pad1.30x1.75mm_HandSolder -> Resistor_SMD:R_0603_1608Metric_Pad0.98x0.95mm_HandSolder
- R7: value 1k -> 220; footprint Resistor_SMD:R_1206_3216Metric_Pad1.30x1.75mm_HandSolder -> Resistor_SMD:R_0603_1608Metric_Pad0.98x0.95mm_HandSolder
- moved Q1 38.4 mm to (109.7, 84.5)
- moved D4 36.5 mm to (117.5, 65.0), turned to 0 degrees
- moved R6 35.3 mm to (87.0, 60.5), turned to 180 degrees
- moved Q2 31.1 mm to (88.5, 51.0), turned to 0 degrees
- moved C10 30.7 mm to (103.0, 70.5), turned to 180 degrees
- moved R7 30.4 mm to (87.0, 73.5), turned to 180 degrees
- moved R3 27.8 mm to (89.0, 44.0)
- moved D3 27.2 mm to (91.0, 72.0), turned to 180 degrees
- moved G2 23.3 mm to (119.5, 65.0)
- moved C7 22.1 mm to (87.0, 41.0)
- moved R2 19.2 mm to (83.5, 76.1), turned to 270 degrees
- moved D5 18.9 mm to (121.1, 65.0), turned to 180 degrees
- moved D6 17.9 mm to (103.0, 65.2)
- moved C2 13.9 mm to (109.5, 76.0)
- moved C1 12.8 mm to (96.5, 76.0)
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Connections:
- C1 pad 1: +5V -> VCC
- C10 pad 1: /EN -> GND
- C10 pad 2: GND -> VCC
- C7 pad 1: GND -> +3V3
- C7 pad 2: +5V -> GND
- C9 pad 1: +3V3 -> /EN
- D1 pad 1: +5V -> VCC
- D2 pad 2: +3V3 -> Net-(D2-Pad2)
- D3 pad 2: +3V3 -> Net-(D2-Pad2)
- D4 pad 2: +3V3 -> Net-(D2-Pad2)
- D5 pad 1: +5V -> Net-(D5-Pad1)
- D5 pad 2: Net-(D5-Pad2) -> Net-(D2-Pad2)
- D6 pad 1: +5V -> VCC
- D6 pad 2: VDD -> Net-(D6-Pad2)
- J1 pad 1: VDD -> +5V
- J1 pad 2: VDD -> +5V
- J1 pad 3: Net-(J1-Pad3) -> GND
- Q1 pad 1: Net-(Q1-Pad1) -> VBUS
- Q1 pad 2: /RTS -> VCC
- Q1 pad 3: /EN -> +5V
- Q2 pad 2: /DTR -> /RTS
- Q2 pad 3: /IO0 -> /EN
- R1 pad 1: Net-(R1-Pad1) -> VBUS
- R1 pad 2: +3V3 -> GND
- R2 pad 1: /LED_TX -> Net-(R2-Pad1)
- R2 pad 2: Net-(D2-Pad1) -> +3V3
- R3 pad 1: /LED_RX -> +3V3
- R3 pad 2: Net-(D3-Pad1) -> /EN
- R4 pad 1: GND -> Net-(Q2-Pad1)
- R4 pad 2: Net-(D4-Pad1) -> /DTR
- R5 pad 1: Net-(Q1-Pad1) -> Net-(Q3-Pad1)
- R5 pad 2: /DTR -> /RTS
- R6 pad 1: Net-(Q2-Pad1) -> /LED_TX
- R6 pad 2: /RTS -> Net-(D2-Pad1)
- R7 pad 1: +3V3 -> /LED_RX
- R7 pad 2: /EN -> Net-(D3-Pad1)
- U1 pad 3: +5V -> VCC
- U2 pad 9: Net-(R1-Pad1) -> Net-(R2-Pad1)
Routing:
- net +3V3: track 159.2 -> 0.00 mm, vias 2 -> 0
- net /D+: track 63.1 -> 0.00 mm
- net /D-: track 60.8 -> 0.00 mm
- net +5V: track 59.0 -> 0.00 mm
- net /RTS: track 43.4 -> 0.00 mm, vias 3 -> 0
- net VBUS: track 43.0 -> 0.00 mm
- net /DTR: track 41.8 -> 0.00 mm, vias 3 -> 0
- net /EN: track 38.4 -> 0.00 mm
- net /MCU_RX: track 36.5 -> 0.00 mm, vias 2 -> 0
- net /MCU_TX: track 35.4 -> 0.00 mm, vias 2 -> 0
- net GND: track 28.2 -> 0.00 mm, vias 32 -> 25
- net /UART_RX: track 27.7 -> 0.00 mm
- net VDD: track 27.6 -> 0.00 mm
- net /LED_RX: track 21.0 -> 0.00 mm
- net /LED_TX: track 21.0 -> 0.00 mm
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- removed copper zone on B.Cu, net GND
- removed copper zone on F.Cu, net GND
Other:
- board size 49 x 63.3 mm -> 48 x 52.5 mm

Commit message: Fixed routing
Parts:
- removed G2: LOGO, Harry:Harry_3
- moved R9 40.0 mm to (89.5, 76.0)
- moved D5 37.8 mm to (88.9, 84.8), turned to 270 degrees
- moved R8 37.0 mm to (86.0, 76.0)
- moved D4 37.0 mm to (86.3, 85.0)
- moved Q2 33.4 mm to (121.5, 56.1)
- moved Q3 33.4 mm to (118.5, 61.1)
- moved R4 33.4 mm to (116.5, 56.1)
- moved R5 33.4 mm to (123.5, 61.1)
- moved R2 18.4 mm to (91.5, 59.5), turned to 180 degrees
- moved R7 12.3 mm to (98.0, 68.0), turned to 270 degrees
- moved C5 11.5 mm to (95.0, 71.5), turned to 180 degrees
- moved D3 9.71 mm to (96.5, 64.0), turned to 270 degrees
- moved C3 9.18 mm to (88.0, 71.5), turned to 180 degrees
- moved R6 7.76 mm to (85.0, 68.0), turned to 270 degrees
- moved C6 7.57 mm to (94.0, 68.5), turned to 180 degrees
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Routing:
- net GND: track 0.00 -> 147.8 mm, vias 25 -> 23
- net +3V3: track 0.00 -> 131.0 mm, vias 0 -> 4
- net /EN: track 0.00 -> 55.8 mm
- net VBUS: track 0.00 -> 45.0 mm
- net /IO0: track 0.00 -> 44.3 mm, vias 1 -> 3
- net VCC: track 0.00 -> 43.2 mm
- net /DTR: track 0.00 -> 40.5 mm, vias 0 -> 2
- net +5V: track 0.00 -> 39.7 mm
- net /RTS: track 0.00 -> 38.2 mm, vias 0 -> 2
- net /D+: track 0.00 -> 34.8 mm
- net Net-(D2-Pad2): track 0.00 -> 33.8 mm, vias 0 -> 3
- net /MCU_RX: track 0.00 -> 33.5 mm, vias 0 -> 2
- net /MCU_TX: track 0.00 -> 32.6 mm, vias 0 -> 2
- net /D-: track 0.00 -> 31.3 mm
- net /HAN_OUT: track 0.00 -> 27.5 mm
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- added copper zone on B.Cu, net GND
- added copper zone on F.Cu, net GND

Commit message: Fixed small issues
Parts:
- moved C5 12.8 mm to (83.0, 67.0), turned to 90 degrees
- moved C3 12.5 mm to (83.0, 60.0), turned to 90 degrees
- moved R7 11.7 mm to (86.5, 70.0), turned to 180 degrees
- moved R6 11.1 mm to (86.5, 57.0), turned to 180 degrees
- moved Q2 8.97 mm to (122.5, 65.0), turned to 90 degrees
- moved R5 8.51 mm to (117.4, 67.0), turned to 0 degrees
- moved C6 8.38 mm to (86.0, 66.0), turned to 90 degrees
- moved C4 8.08 mm to (86.0, 61.0), turned to 270 degrees
- moved D3 7.50 mm to (90.5, 68.5), turned to 180 degrees
- moved R4 7.15 mm to (122.5, 60.0), turned to 0 degrees
- moved D2 6.80 mm to (90.5, 58.5), turned to 180 degrees
- moved R2 5.66 mm to (95.5, 63.5), turned to 90 degrees
- moved R9 2.00 mm to (87.5, 76.0)
- moved C7 1.50 mm to (87.0, 45.0)
- moved C8 1.50 mm to (85.0, 48.0)
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Routing:
- net GND: track 147.8 -> 55.1 mm, vias 23 -> 43
- net /IO0: track 44.3 -> 6.77 mm, vias 3 -> 0
- net +3V3: track 131.0 -> 118.7 mm
- net /LED_RX: track 16.0 -> 7.83 mm, vias 0 -> 2
- net VCC: track 43.2 -> 50.2 mm
- net /EN: track 55.8 -> 51.3 mm, vias 0 -> 2
- net /UART_RX: track 16.6 -> 12.5 mm
- net /D+: track 34.8 -> 31.2 mm, vias 0 -> 2
- net /RTS: track 38.2 -> 41.7 mm, vias 2 -> 0
- net /MCU_TX: track 32.6 -> 29.7 mm, vias 2 -> 0
- net +5V: track 39.7 -> 42.5 mm
- net /D-: track 31.3 -> 28.9 mm, vias 0 -> 2
- net Net-(D2-Pad2): track 33.8 -> 31.5 mm, vias 3 -> 2
- net Net-(Q2-Pad1): track 4.27 -> 6.52 mm
- net /DTR: track 40.5 -> 39.0 mm, vias 2 -> 3
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
Commit message: Updates
Parts:
- moved R7 12.2 mm to (97.3, 64.4), turned to 270 degrees
- moved D2 11.8 mm to (95.1, 69.3), turned to 270 degrees
- moved R6 11.3 mm to (95.1, 64.4), turned to 270 degrees
- moved R2 9.48 mm to (88.0, 69.3), turned to 270 degrees
- moved R4 8.68 mm to (118.3, 67.6), turned to 180 degrees
- moved R5 7.29 mm to (122.3, 61.6)
- moved R1 7.11 mm to (92.1, 69.3)
- moved D3 6.96 mm to (97.4, 69.3), turned to 270 degrees
- moved R8 3.95 mm to (81.6, 75.4)
- moved R9 3.65 mm to (83.9, 75.4)
- moved C3 2.94 mm to (82.1, 62.8)
- moved C4 2.71 mm to (84.9, 63.5), turned to 90 degrees
- moved R11 2.54 mm to (121.0, 50.5)
- moved R12 2.54 mm to (119.0, 50.5), turned to 90 degrees
- moved C6 2.10 mm to (84.9, 67.8)
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Connections:
- D2 pad 2: Net-(D2-Pad2) -> +3V3
- D3 pad 2: Net-(D2-Pad2) -> +3V3
- D4 pad 2: Net-(D2-Pad2) -> +3V3
- D5 pad 2: Net-(D2-Pad2) -> +3V3
- D6 pad 2: Net-(D6-Pad2) -> (no net)
- J1 pad 4: Net-(J1-Pad4) -> (no net)
- M1 pad 4: Net-(M1-Pad4) -> (no net)
- U2 pad 1: Net-(U2-Pad1) -> (no net)
- U2 pad 10: Net-(U2-Pad10) -> (no net)
- U2 pad 11: Net-(U2-Pad11) -> (no net)
- U2 pad 12: Net-(U2-Pad12) -> (no net)
- U2 pad 15: Net-(U2-Pad15) -> (no net)
- U2 pad 16: Net-(U2-Pad16) -> (no net)
- U2 pad 17: Net-(U2-Pad17) -> (no net)
- U2 pad 18: Net-(U2-Pad18) -> (no net)
- U2 pad 22: Net-(U2-Pad22) -> (no net)
- U2 pad 24: Net-(U2-Pad24) -> (no net)
- U2 pad 25: GND -> (no net)
- U3 pad 10: Net-(U3-Pad10) -> (no net)
- U3 pad 11: Net-(U3-Pad11) -> (no net)
- U3 pad 12: Net-(U3-Pad12) -> (no net)
- U3 pad 13: Net-(U3-Pad13) -> (no net)
- U3 pad 14: Net-(U3-Pad14) -> (no net)
- U3 pad 17: Net-(U3-Pad17) -> (no net)
- U3 pad 18: Net-(U3-Pad18) -> (no net)
- U3 pad 19: Net-(U3-Pad19) -> (no net)
- U3 pad 20: Net-(U3-Pad20) -> (no net)
- U3 pad 21: Net-(U3-Pad21) -> (no net)
- U3 pad 22: Net-(U3-Pad22) -> (no net)
- U3 pad 23: Net-(U3-Pad23) -> (no net)
- U3 pad 24: Net-(U3-Pad24) -> (no net)
- U3 pad 26: Net-(U3-Pad26) -> (no net)
- U3 pad 28: Net-(U3-Pad28) -> (no net)
- U3 pad 29: Net-(U3-Pad29) -> (no net)
- U3 pad 30: Net-(U3-Pad30) -> (no net)
- U3 pad 31: Net-(U3-Pad31) -> (no net)
- U3 pad 32: Net-(U3-Pad32) -> (no net)
- U3 pad 33: Net-(U3-Pad33) -> (no net)
- U3 pad 36: Net-(U3-Pad36) -> (no net)
- U3 pad 37: Net-(U3-Pad37) -> (no net)
- U3 pad 39: GND -> (no net)
- U3 pad 4: Net-(U3-Pad4) -> (no net)
- U3 pad 5: Net-(U3-Pad5) -> (no net)
- U3 pad 6: Net-(U3-Pad6) -> (no net)
- U3 pad 7: Net-(U3-Pad7) -> (no net)
- U3 pad 8: Net-(U3-Pad8) -> (no net)
- U3 pad 9: Net-(U3-Pad9) -> (no net)
Routing:
- net GND: track 55.1 -> 5.69 mm, vias 43 -> 48
- net Net-(D2-Pad2): track 31.5 -> 0.00 mm, vias 2 -> 0
- net +3V3: track 118.7 -> 145.0 mm, vias 4 -> 5
- net /LED_TX: track 13.2 -> 3.42 mm, vias 2 -> 0
- net VCC: track 50.2 -> 40.8 mm
- net /D+: track 31.2 -> 40.5 mm, vias 2 -> 0
- net /D-: track 28.9 -> 36.3 mm, vias 2 -> 0
- net /RTS: track 41.7 -> 46.9 mm
- net VBUS: track 46.5 -> 51.6 mm, vias 0 -> 2
- net /MCU_RX: track 33.7 -> 28.8 mm
- net Net-(D3-Pad1): track 7.56 -> 3.20 mm
- net Net-(Q2-Pad1): track 6.52 -> 2.34 mm
- net /DTR: track 39.0 -> 35.5 mm, vias 3 -> 2
- net Net-(D2-Pad1): track 6.50 -> 3.18 mm
- net Net-(R2-Pad1): track 6.65 -> 3.71 mm
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
Commit message: New gerber files
Routing:
- net GND: vias 48 -> 47
Other:
- rule pad_to_mask_clearance: 0.2 -> 0
