File: AidonBoard32.kicad_pcb (KiCad board)
At the start: 2 copper layers, 48 x 52.5 mm, 38 parts, among them J1 RJ12, M1 U-F-M5DD-Y-L, Q1 Si2301CDS-T1-GE3, Q2 MMBT3904, Q3 MMBT3904, Q4 MMBT3904, U1 AMS1117-3V3, U2 CP2102N-GQFN24, U3 ESP32-WROOM

Commit message: Fix
Parts:
- moved D4 0.19 mm to (85.3, 84.8), turned to 180 degrees
- moved D3 0.08 mm to (97.3, 69.3)
Connections:
- D6 pad 2: (no net) -> Net-(D6-Pad2)
- J1 pad 4: (no net) -> Net-(J1-Pad4)
- M1 pad 4: (no net) -> Net-(M1-Pad4)
- U2 pad 1: (no net) -> Net-(U2-Pad1)
- U2 pad 10: (no net) -> Net-(U2-Pad10)
- U2 pad 11: (no net) -> Net-(U2-Pad11)
- U2 pad 12: (no net) -> Net-(U2-Pad12)
- U2 pad 15: (no net) -> Net-(U2-Pad15)
- U2 pad 16: (no net) -> Net-(U2-Pad16)
- U2 pad 17: (no net) -> Net-(U2-Pad17)
- U2 pad 18: (no net) -> Net-(U2-Pad18)
- U2 pad 22: (no net) -> Net-(U2-Pad22)
- U2 pad 24: (no net) -> Net-(U2-Pad24)
- U2 pad 25: (no net) -> Net-(U2-Pad25)
- U3 pad 10: (no net) -> Net-(U3-Pad10)
- U3 pad 11: (no net) -> Net-(U3-Pad11)
- U3 pad 12: (no net) -> Net-(U3-Pad12)
- U3 pad 13: (no net) -> Net-(U3-Pad13)
- U3 pad 14: (no net) -> Net-(U3-Pad14)
- U3 pad 17: (no net) -> Net-(U3-Pad17)
- U3 pad 18: (no net) -> Net-(U3-Pad18)
- U3 pad 19: (no net) -> Net-(U3-Pad19)
- U3 pad 20: (no net) -> Net-(U3-Pad20)
- U3 pad 21: (no net) -> Net-(U3-Pad21)
- U3 pad 22: (no net) -> Net-(U3-Pad22)
- U3 pad 23: (no net) -> Net-(U3-Pad23)
- U3 pad 24: (no net) -> Net-(U3-Pad24)
- U3 pad 26: (no net) -> Net-(U3-Pad26)
- U3 pad 28: (no net) -> Net-(U3-Pad28)
- U3 pad 29: (no net) -> Net-(U3-Pad29)
- U3 pad 30: (no net) -> Net-(U3-Pad30)
- U3 pad 31: (no net) -> Net-(U3-Pad31)
- U3 pad 32: (no net) -> Net-(U3-Pad32)
- U3 pad 33: (no net) -> Net-(U3-Pad33)
- U3 pad 36: (no net) -> Net-(U3-Pad36)
- U3 pad 37: (no net) -> Net-(U3-Pad37)
- U3 pad 39: (no net) -> Net-(U3-Pad39)
- U3 pad 4: (no net) -> Net-(U3-Pad4)
- U3 pad 5: (no net) -> Net-(U3-Pad5)
- U3 pad 6: (no net) -> Net-(U3-Pad6)
- U3 pad 7: (no net) -> Net-(U3-Pad7)
- U3 pad 8: (no net) -> Net-(U3-Pad8)
- U3 pad 9: (no net) -> Net-(U3-Pad9)
Routing:
- net Net-(D4-Pad1): track 9.28 -> 10.5 mm
